File: RFIDr_Open_Top.kicad_pcb (KiCad board)
At the start: 4 copper layers, 188.5 x 34 mm, 522 parts, among them P1 CONN_01X04, P2 CONN_02X04, P3 CONN_02X08, P4 CONN_02X05, P5 CONN_02X08, Q1 DMP2305, Q2 CTRL_NMOS, SW1 SW_RESET, SW2 SW_SAMPLE, SW3 SW_RESET, SW4 SW_SAMPLE, U1 USB_Micro_B, U10 10M02E144, U11 TSV358, U12 BatJSTCnctr, U13 Thermocouple, U14 BQ24073, U15 AP7361C-Y5-13, U16 AP7361C-Y5-13, U17 AP7361C-Y5-13, U18 SMA_72970, U19 SMA_72970, U2 PUSB2X4Y, U20 J0910CF15B0100, U21 HHM22106, U22 SKY13350, U23 SMA_72970, U24 MAX2204, U25 SG210STF_XO, U26 CX3225GB_36MHz_XTAL, U27 SKY65111, U28 SX1257, U29 PE64906, U3 NLAS5223B, U30 PE64102, U31 PE64906, U32 PE64102, U33 PAT1220, U34 MountingHole, U35 MountingHole, U36 MountingHole, U37 MountingHole, U38 MountingHole, U39 SF2049E, U4 FC-135_32p768_XTAL, U40 LP5951MF, U41 0917BL18B100E, U42 LTC5505-1, U43 LM2767M5, U44 MBR0520LTR, U45 SN74LV1T34, U46 LP3985IM5-5.0, U47 SN74LV1T34, U5 DMN63D8LDW-7, U6 NRF51822, U7 NX2520SA_16MHz_XTAL, U8 NLAS5223B, U9 NLAS5223B

Commit message: DNI C67 In Schematics and Layout
C67 was DNIed in the BOM but not in the schematics/layout. C67 needs to be DNI or a small value for the SX1257 DAC autocalibration procedure to work. We DNIed C67 in both the schematic and layout to eliminate confusion.
Parts:
- C67: value 100n -> DNI
Changed lines of the file:
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@@
     (add_net /ANT1)
     (add_net /CHGB)
+    (add_net /CTRLR_CIPO)
+    (add_net /CTRLR_COPI_CAP0_RDIO)
+    (add_net /CTRLR_COPI_CAP1)
+    (add_net /CTRLR_COPI_CAP2)
+    (add_net /CTRLR_COPI_CAP3)
+    (add_net /CTRLR_NPS_DTC)
+    (add_net /CTRLR_NPS_RDIO)
+    (add_net /CTRLR_PCLK)
     (add_net /DIO2)
     (add_net /DIO3)
@@
     (add_net /FPGA_OUT_I)
     (add_net /FPGA_OUT_Q)
-    (add_net /CTRLR_CIPO)
-    (add_net /CTRLR_COPI_CAP0_RDIO)
-    (add_net /CTRLR_COPI_CAP1)
-    (add_net /CTRLR_COPI_CAP2)
-    (add_net /CTRLR_COPI_CAP3)
-    (add_net /CTRLR_NPS_DTC)
-    (add_net /CTRLR_NPS_RDIO)
-    (add_net /CTRLR_PCLK)
     (add_net /OPA_SPDT1_CTL)
     (add_net /PGOODB)
@@
     (add_net /RFIDr_Open_DigBB/CYCLE)
     (add_net /RFIDr_Open_DigBB/FPGA_IRQ)
-    (add_net /RFIDr_Open_DigBB/FPGA_RST_N)
     (add_net /RFIDr_Open_DigBB/FPGA_PRPHL_CIPO)
     (add_net /RFIDr_Open_DigBB/FPGA_PRPHL_COPI)
     (add_net /RFIDr_Open_DigBB/FPGA_PRPHL_NPS)
     (add_net /RFIDr_Open_DigBB/FPGA_PRPHL_PCLK)
+    (add_net /RFIDr_Open_DigBB/FPGA_RST_N)
     (add_net /RFIDr_Open_DigBB/FPGA_TCK_MCU)
     (add_net /RFIDr_Open_DigBB/FPGA_TDI_MCU)
@@
       (effects (font (size 0.5 0.5) (thickness 0.1)))
     )
-    (fp_text value 100n (at 0 1.7 180) (layer F.Fab)
-      (effects (font (size 1 1) (thickness 0.15)))
-    )
+    (fp_text value DNI (at 0 1.7 180) (layer F.Fab)
+      (effects (font (size 1 1) (thickness 0.15)))
+    )

Commit message: Change value of C126 to 1nF.
In order for the DAC autocalibration routine to work, C67 needs to be DNI and C126 needs to be 1nF. Previously this had been changed in the BOM but not in the schematic or PCB. We fix this here.
Parts:
- C126: value 100n -> 1n
Changed lines of the file:
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@@
       (effects (font (size 0.5 0.5) (thickness 0.1)))
     )
-    (fp_text value 100n (at 0 1.7) (layer F.Fab)
+    (fp_text value 1n (at 0 1.7) (layer F.Fab)
       (effects (font (size 1 1) (thickness 0.15)))
     )
